Commit message: small adjustmrnts

File: config/urdf/arm.urdf (robot description, URDF)
Before this commit: robot test_robot, 5 links, 4 joints
Joints:
- joint joint3: child link5 -> link4
- joint joint4: child link4 -> link5; parent link5 -> link4

File: config/urdf/tool.urdf (robot description, URDF)
Before this commit: robot test_robot, 5 links, 4 joints
Joints:
- joint joint2: child link5 -> link4
- joint joint3: child link4 -> link5; parent link5 -> link4
